File: 0037_SD_Card_Module_Classic.kicad_sch (KiCad schematic)
At the start: 6 parts, among them IC1 74LVC125APW,118, J1 Micro_SD

Commit message: Add files via upload
Parts:
- added D1: LED, LED_SMD:LED_0603_1608Metric, symbol Device:LED
- added R5: 470r, Resistor_SMD:R_0603_1608Metric, symbol Device:R
- added U1: ~, Moduler_:pin_header, symbol moduler_pin:air
- IC1: footprint SOP65P640X110-14N -> 74LVC125APW:SOP65P640X110-14N
- J1: footprint L-KLS1-TF-003-H1.85-R -> meminle:L-KLS1-TF-003-H1.85-R
- R1, R2, R3, R4: footprint (none) -> Resistor_SMD:R_0603_1608Metric
Connections:
- net +3V3: now also R5.1, U1.8
- net CS: now also U1.3
- net GND: now also J1.10 (G_1), J1.11 (G_2), J1.12 (G_3), J1.13 (G_4), D1.1 (K), U1.9
- net MISO: now also U1.2
- net MOSI: now also U1.1
- net SCK: now also U1.4
- new net: D1.2 (A), R5.2
- no-connect marks 3 -> 15
Other:
- note added: "AIR PIN"
- note added: "SENSOR"
- moved on the sheet: IC1, J1, R1, R2, R4
